File: Circuits/MoterController/OreoMotorController/_autosave-OreoMotorController.sch (KiCad schematic (older format))
At the start: 20 parts

Commit message: refactor : finished circuit design
Parts:
- removed J?: Conn_01x02_Female, symbol Connector:Conn_01x02_Female
- added D2: 1N5822, symbol Diode:1N5822
- added J3: Power, symbol Connector:Conn_01x02_Male
- added SW1: SW_SPDT, symbol Switch:SW_SPDT
- 100mF1: renamed from C?; footprint (none) -> Capacitor_THT:CP_Radial_D12.5mm_P5.00mm
- A1: renamed from A?; footprint Module:Arduino_Nano -> (none)
- R1, R2: renamed from R?; value R -> 330
- U2: renamed from U?; footprint Package_TO_SOT_SMD:TO-263-5_TabPin3 -> (none)
- gave numbers to parts that had none: 14
Connections:
- wire segments 107 -> 125
- no-connect marks 9 -> 17
